File: encoder/sturcde/sturcde.kicad_sch (KiCad schematic)
At the start: 10 parts, among them J1 Left A, J2 Left B, J3 Left Encoder, J4 Right A, J5 Right B, J6 Right Encoder

Commit message: Add logo; general cleanups and prep for pcbway.
Other:
- company: (none) -> Astoria HS Riverbots FRC #6845
- title: (none) -> The Stupid Ridiculously-Cheap Drive Encoder
Changed lines of the file:
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@@
 (kicad_sch (version 20230121) (generator eeschema)
-  (paper "A4")
+  (paper "USLetter")
+  (title_block
+    (title "The Stupid Ridiculously-Cheap Drive Encoder")
+    (date "2024-02-14")
+    (rev "1.0")
+    (company "Astoria HS Riverbots FRC #6845")
+  )
   (junction (at 120.65 49.53) (diameter 0) (color 0 0 0 0)
   )
